File: LRUs/User Control Unit/Electrical/User Control Board/user_control_board/3V3.kicad_sch (KiCad schematic)
At the start: 7 parts, among them U17 AMS1117-3.3

Commit message: connectors and 5v buck partially done
Parts:
- C10: renamed from C61; footprint valve_pcb_footprints:C_0805_2012Metric -> Capacitor_SMD:C_0805_2012Metric
- C11: renamed from C63; footprint valve_pcb_footprints:C_0805_2012Metric -> Capacitor_SMD:C_0805_2012Metric
- R18: renamed from R242; footprint valve_pcb_footprints:R_0603_1608Metric -> Resistor_SMD:R_0603_1608Metric
- renumbered C65 to C12, D42 to D2, TP107 to TP7, U17 to U3
Changed lines of the file:
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@@
 		(dnp no)
 		(fields_autoplaced yes)
-		(property "Reference" "U17"
+		(property "Reference" "U3"
 			(at 142.24 85.09 0)
 			(show_name no)
@@
 			(project "user_control_board"
 				(path "/4e4fbe8c-7357-4f75-8a99-a243261c2770/41704214-6d9d-43c3-b829-66d009a1b449"
-					(reference "U17")
+					(reference "U3")
 					(unit 1)
 				)
@@
 		(dnp no)
 		(fields_autoplaced yes)
-		(property "Reference" "#PWR0170"
+		(property "Reference" "#PWR032"
 			(at 162.56 106.68 0)
 			(hide yes)
@@
 			(project "user_control_board"
 				(path "/4e4fbe8c-7357-4f75-8a99-a243261c2770/41704214-6d9d-43c3-b829-66d009a1b449"
-					(reference "#PWR0170")
+					(reference "#PWR032")
 					(unit 1)
 				)
@@
 		(dnp no)
 		(fields_autoplaced yes)
-		(property "Reference" "#PWR0172"
+		(property "Reference" "#PWR033"
 			(at 175.26 106.68 0)
 			(hide yes)
@@
 			(project "user_control_board"
 				(path "/4e4fbe8c-7357-4f75-8a99-a243261c2770/41704214-6d9d-43c3-b829-66d009a1b449"
-					(reference "#PWR0172")
+					(reference "#PWR033")
 					(unit 1)
 				)
@@
 		(dnp no)
 		(fields_autoplaced yes)
-		(property "Reference" "#PWR0168"
+		(property "Reference" "#PWR031"
 			(at 142.24 106.68 0)
 			(hide yes)
@@
 			(project "user_control_board"
 				(path "/4e4fbe8c-7357-4f75-8a99-a243261c2770/41704214-6d9d-43c3-b829-66d009a1b449"
-					(reference "#PWR0168")
+					(reference "#PWR031")
 					(unit 1)
 				)
@@
 		(dnp no)
 		(fields_autoplaced yes)
-		(property "Reference" "#PWR0163"
+		(property "Reference" "#PWR030"
 			(at 119.38 106.68 0)
 			(hide yes)
@@
 			(project "user_control_board"
 				(path "/4e4fbe8c-7357-4f75-8a99-a243261c2770/41704214-6d9d-43c3-b829-66d009a1b449"
-					(reference "#PWR0163")
+					(reference "#PWR030")
 					(unit 1)
 				)
@@
 		(in_pos_files yes)
 		(dnp no)
-		(property "Reference" "C61"
+		(property "Reference" "C10"
 			(at 121.158 94.234 0)
 			(show_name no)
@@
 			)
 		)
-		(property "Footprint" "valve_pcb_footprints:C_0805_2012Metric"
+		(property "Footprint" "Capacitor_SMD:C_0805_2012Metric"
 			(at 119.38 96.52 0)
 			(hide yes)
@@
 			(project "user_control_board"
 				(path "/4e4fbe8c-7357-4f75-8a99-a243261c2770/41704214-6d9d-43c3-b829-66d009a1b449"
-					(reference "C61")
+					(reference "C10")
 					(unit 1)
 				)
@@
 		(in_pos_files yes)
 		(dnp no)
-		(property "Reference" "C63"
+		(property "Reference" "C11"
 			(at 164.084 94.234 0)
 			(show_name no)
@@
 			)
 		)
-		(property "Footprint" "valve_pcb_footprints:C_0805_2012Metric"
+		(property "Footprint" "Capacitor_SMD:C_0805_2012Metric"
 			(at 162.56 96.52 0)
 			(hide yes)
@@
 			(project "user_control_board"
 				(path "/4e4fbe8c-7357-4f75-8a99-a243261c2770/41704214-6d9d-43c3-b829-66d009a1b449"
-					(reference "C63")
+					(reference "C11")
 					(unit 1)
 				)
@@
 		(dnp no)
 		(fields_autoplaced yes)
-		(property "Reference" "#FLG05"
+		(property "Reference" "#FLG02"
 			(at 127 89.535 0)
 			(hide yes)
@@
 			(project "user_control_board"
 				(path "/4e4fbe8c-7357-4f75-8a99-a243261c2770/41704214-6d9d-43c3-b829-66d009a1b449"
-					(reference "#FLG05")
+					(reference "#FLG02")
 					(unit 1)
 				)
@@
 		(dnp no)
 		(fields_autoplaced yes)
-		(property "Reference" "#PWR0318"
+		(property "Reference" "#PWR034"
 			(at 189.23 121.92 0)
 			(hide yes)
@@
 			(project "user_control_board"
 				(path "/4e4fbe8c-7357-4f75-8a99-a243261c2770/41704214-6d9d-43c3-b829-66d009a1b449"
-					(reference "#PWR0318")
+					(reference "#PWR034")
 					(unit 1)
 				)
@@
 		(in_pos_files yes)
 		(dnp no)
-		(property "Reference" "R242"
+		(property "Reference" "R18"
 			(at 193.294 96.52 0)
 			(show_name no)
@@
 			)
 		)
-		(property "Footprint" "valve_pcb_footprints:R_0603_1608Metric"
+		(property "Footprint" "Resistor_SMD:R_0603_1608Metric"
 			(at 189.23 99.06 0)
 			(hide yes)
@@
 			(project "user_control_board"
 				(path "/4e4fbe8c-7357-4f75-8a99-a243261c2770/41704214-6d9d-43c3-b829-66d009a1b449"
-					(reference "R242")
+					(reference "R18")
 					(unit 1)
 				)
@@
 		(in_pos_files yes)
 		(dnp no)
-		(property "Reference" "D42"
+		(property "Reference" "D2"
 			(at 191.77 107.442 90)
 			(show_name no)
@@
 			(project "user_control_board"
 				(path "/4e4fbe8c-7357-4f75-8a99-a243261c2770/41704214-6d9d-43c3-b829-66d009a1b449"
-					(reference "D42")
+					(reference "D2")
 					(unit 1)
 				)
@@
 		(in_pos_files yes)
 		(dnp no)
-		(property "Reference" "C65"
+		(property "Reference" "C12"
 			(at 177.038 94.488 0)
 			(show_name no)
@@
 			(project "user_control_board"
 				(path "/4e4fbe8c-7357-4f75-8a99-a243261c2770/41704214-6d9d-43c3-b829-66d009a1b449"
-					(reference "C65")
+					(reference "C12")
 					(unit 1)
 					(variant
@@
 		(in_pos_files yes)
 		(dnp no)
-		(property "Reference" "TP107"
+		(property "Reference" "TP7"
 			(at 176.53 88.9 90)
 			(show_name no)
@@
 			(project "user_control_board"
 				(path "/4e4fbe8c-7357-4f75-8a99-a243261c2770/41704214-6d9d-43c3-b829-66d009a1b449"
-					(reference "TP107")
+					(reference "TP7")
 					(unit 1)
 				)
