File: LRUs/User Control Unit/Electrical/User Control Board/user_control_board/5v.kicad_sch (KiCad schematic)
At the start: 24 parts, among them U1 TPS62933P

Commit message: connectors and 5v buck partially done
Parts:
- C5: renamed from C3; footprint valve_pcb_footprints:C_0402_1005Metric -> Capacitor_SMD:C_01005_0402Metric
- C6: renamed from C4; footprint valve_pcb_footprints:C_0402_1005Metric -> Capacitor_SMD:C_0402_1005Metric
- C7: renamed from C5; footprint valve_pcb_footprints:C_0402_1005Metric -> Capacitor_SMD:C_0402_1005Metric
- R10: renamed from R2; footprint valve_pcb_footprints:R_0603_1608Metric -> Resistor_SMD:R_0603_1608Metric
- R11: renamed from R3; footprint valve_pcb_footprints:R_0603_1608Metric -> Resistor_SMD:R_0603_1608Metric
- R12: renamed from R4; footprint valve_pcb_footprints:R_0603_1608Metric -> Resistor_SMD:R_0603_1608Metric
- R13: renamed from R5; footprint valve_pcb_footprints:R_0603_1608Metric -> Resistor_SMD:R_0603_1608Metric
- R14: renamed from R6; footprint valve_pcb_footprints:R_0603_1608Metric -> Resistor_SMD:R_0603_1608Metric
- R15: renamed from R7; footprint valve_pcb_footprints:R_0603_1608Metric -> Resistor_SMD:R_0603_1608Metric
- R16: renamed from R8; footprint valve_pcb_footprints:R_0603_1608Metric -> Resistor_SMD:R_0603_1608Metric
- R17: renamed from R9; footprint valve_pcb_footprints:R_0603_1608Metric -> Resistor_SMD:R_0603_1608Metric
- R9: renamed from R1; footprint valve_pcb_footprints:R_0603_1608Metric -> Resistor_SMD:R_0603_1608Metric
- renumbered C1 to C3, C2 to C4, C6 to C8, C7 to C9, TP1 to TP2, TP2 to TP3, TP3 to TP4, TP4 to TP5, TP5 to TP6, U1 to U2
Connections:
- net SW: now also L1.2; no longer L1.1
- net VOUT: now also L1.1; no longer L1.2
- no-connect marks 0 -> 1
Other:
- moved on the sheet: L1
