File: LRUs/User Control Unit/Electrical/User Control Board/user_control_board/mechanicak.kicad_sch (KiCad schematic)
At the start: 4 parts

Commit message: connectors and 5v buck partially done
Parts:
- renumbered H3 to H2, H2 to H3
Changed lines of the file:
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@@
 		(dnp no)
 		(fields_autoplaced yes)
-		(property "Reference" "#PWR091"
+		(property "Reference" "#PWR047"
 			(at 137.16 92.71 0)
 			(hide yes)
@@
 			(project "user_control_board"
 				(path "/5b97fe44-b582-48d0-85a5-3f832c28b8e4"
-					(reference "#PWR091")
+					(reference "#PWR047")
 					(unit 1)
 				)
@@
 		(dnp no)
 		(fields_autoplaced yes)
-		(property "Reference" "H2"
+		(property "Reference" "H3"
 			(at 139.7 68.5799 0)
 			(show_name no)
@@
 			(project "user_control_board"
 				(path "/5b97fe44-b582-48d0-85a5-3f832c28b8e4"
-					(reference "H2")
+					(reference "H3")
 					(unit 1)
 				)
@@
 		(dnp no)
 		(fields_autoplaced yes)
-		(property "Reference" "#PWR090"
+		(property "Reference" "#PWR045"
 			(at 111.76 92.71 0)
 			(hide yes)
@@
 			(project "user_control_board"
 				(path "/5b97fe44-b582-48d0-85a5-3f832c28b8e4"
-					(reference "#PWR090")
+					(reference "#PWR045")
 					(unit 1)
 				)
@@
 		(dnp no)
 		(fields_autoplaced yes)
-		(property "Reference" "H3"
+		(property "Reference" "H2"
 			(at 114.3 81.2799 0)
 			(show_name no)
@@
 			(project "user_control_board"
 				(path "/5b97fe44-b582-48d0-85a5-3f832c28b8e4"
-					(reference "H3")
+					(reference "H2")
 					(unit 1)
 				)
@@
 		(dnp no)
 		(fields_autoplaced yes)
-		(property "Reference" "#PWR088"
+		(property "Reference" "#PWR044"
 			(at 111.76 80.01 0)
 			(hide yes)
@@
 			(project "user_control_board"
 				(path "/5b97fe44-b582-48d0-85a5-3f832c28b8e4"
-					(reference "#PWR088")
+					(reference "#PWR044")
 					(unit 1)
 				)
@@
 		(dnp no)
 		(fields_autoplaced yes)
-		(property "Reference" "#PWR089"
+		(property "Reference" "#PWR046"
 			(at 137.16 80.01 0)
 			(hide yes)
@@
 			(project "user_control_board"
 				(path "/5b97fe44-b582-48d0-85a5-3f832c28b8e4"
-					(reference "#PWR089")
-					(unit 1)
-				)
+					(reference "#PWR046")
+					(unit 1)
+				)
