File: LRUs/User Control Unit/Electrical/User Control Board/user_control_board/sd_card.kicad_sch (KiCad schematic)
At the start: 13 parts, among them J16 Micro_SD_Card_Det2, U32 TPD6E05U06RVZ

Commit message: need to run DCR
Connections:
- net SDMMC1_CK renamed GP18
- net SDMMC1_D0 renamed GP16
- net SDMMC1_D1 renamed GP19
- net SDMMC1_D3 renamed GP7
Changed lines of the file:
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@@
+	)
+	(junction
+		(at 68.58 99.06)
+		(diameter 0)
+		(color 0 0 0 0)
 	)
 	(junction
@@
 	)
 	(junction
+		(at 78.74 111.76)
+		(diameter 0)
+		(color 0 0 0 0)
+	)
+	(junction
+		(at 93.98 106.68)
+		(diameter 0)
+		(color 0 0 0 0)
+	)
+	(junction
 		(at 162.56 111.76)
 		(diameter 0)
@@
 	(junction
 		(at 149.86 63.5)
+		(diameter 0)
+		(color 0 0 0 0)
+	)
+	(junction
+		(at 87.63 114.3)
 		(diameter 0)
 		(color 0 0 0 0)
@@
 	(wire
 		(pts
+			(xy 92.71 74.93) (xy 93.98 74.93)
+		)
+		(stroke
+			(width 0)
+			(type default)
+		)
+	)
+	(wire
+		(pts
 			(xy 194.31 121.92) (xy 194.31 119.38)
 		)
@@
 	(wire
 		(pts
-			(xy 49.53 106.68) (xy 111.76 106.68)
+			(xy 49.53 106.68) (xy 93.98 106.68)
 		)
 		(stroke
@@
 	(wire
 		(pts
+			(xy 78.74 83.82) (xy 78.74 111.76)
+		)
+		(stroke
+			(width 0)
+			(type default)
+		)
+	)
+	(wire
+		(pts
 			(xy 160.02 73.66) (xy 160.02 76.2)
 		)
@@
 	(wire
 		(pts
-			(xy 49.53 114.3) (xy 102.87 114.3)
+			(xy 49.53 114.3) (xy 87.63 114.3)
 		)
 		(stroke
@@
 	(wire
 		(pts
+			(xy 87.63 83.82) (xy 87.63 114.3)
+		)
+		(stroke
+			(width 0)
+			(type default)
+		)
+	)
+	(wire
+		(pts
+			(xy 93.98 106.68) (xy 111.76 106.68)
+		)
+		(stroke
+			(width 0)
+			(type default)
+		)
+	)
+	(wire
+		(pts
+			(xy 93.98 74.93) (xy 93.98 106.68)
+		)
+		(stroke
+			(width 0)
+			(type default)
+		)
+	)
+	(wire
+		(pts
 			(xy 242.57 121.92) (xy 242.57 119.38)
 		)
@@
 	(wire
 		(pts
+			(xy 68.58 83.82) (xy 68.58 99.06)
+		)
+		(stroke
+			(width 0)
+			(type default)
+		)
+	)
+	(wire
+		(pts
+			(xy 77.47 83.82) (xy 78.74 83.82)
+		)
+		(stroke
+			(width 0)
+			(type default)
+		)
+	)
+	(wire
+		(pts
 			(xy 147.32 99.06) (xy 196.85 99.06)
 		)
@@
 		(pts
 			(xy 49.53 111.76) (xy 111.76 111.76)
+		)
+		(stroke
+			(width 0)
+			(type default)
+		)
+	)
+	(wire
+		(pts
+			(xy 67.31 83.82) (xy 68.58 83.82)
+		)
+		(stroke
+			(width 0)
+			(type default)
+		)
+	)
+	(wire
+		(pts
+			(xy 87.63 114.3) (xy 102.87 114.3)
 		)
 		(stroke
@@
 			)
 			(justify right bottom)
+		)
+	)
+	(global_label "GP19"
+		(shape input)
+		(at 87.63 83.82 180)
+		(fields_autoplaced yes)
+		(effects
+			(font
+				(size 1.27 1.27)
+			)
+			(justify right)
+		)
+		(property "Intersheetrefs" "${INTERSHEET_REFS}"
+			(at 79.6858 83.82 0)
+			(hide yes)
+			(show_name no)
+			(do_not_autoplace no)
+			(effects
+				(font
+					(size 1.27 1.27)
+				)
+				(justify right)
+			)
 		)
 	)
@@
 			(hide yes)
 			(show_name no)
+			(do_not_autoplace no)
+			(effects
+				(font
+					(size 1.27 1.27)
+				)
+				(justify right)
+			)
+		)
+	)
+	(global_label "GP16"
+		(shape input)
+		(at 77.47 83.82 180)
+		(fields_autoplaced yes)
+		(effects
+			(font
+				(size 1.27 1.27)
+			)
+			(justify right)
+		)
+		(property "Intersheetrefs" "${INTERSHEET_REFS}"
+			(at 69.5258 83.82 0)
+			(hide yes)
+			(show_name no)
+			(do_not_autoplace no)
+			(effects
+				(font
+					(size 1.27 1.27)
+				)
+				(justify right)
+			)
+		)
+	)
+	(global_label "GP18"
+		(shape input)
+		(at 92.71 74.93 180)
+		(fields_autoplaced yes)
+		(effects
+			(font
+				(size 1.27 1.27)
+			)
+			(justify right)
+		)
+		(property "Intersheetrefs" "${INTERSHEET_REFS}"
+			(at 84.7658 74.93 0)
+			(hide yes)
+			(show_name no)
+			(do_not_autoplace no)
+			(effects
+				(font
+					(size 1.27 1.27)
+				)
+				(justify right)
+			)
+		)
+	)
+	(global_label "GP7"
+		(shape input)
+		(at 67.31 83.82 180)
+		(fields_autoplaced yes)
+		(effects
+			(font
+				(size 1.27 1.27)
+			)
+			(justify right)
+		)
+		(property "Intersheetrefs" "${INTERSHEET_REFS}"
+			(at 60.5753 83.82 0)
+			(hide yes)
+			(show_name no)

Commit message: connectors and 5v buck partially done
Parts:
- removed R165, R167, R168: 0, valve_pcb_footprints:R_0603_1608Metric, symbol Device:R_Small_US
- C1: renamed from C107; footprint valve_pcb_footprints:C_0805_2012Metric -> Capacitor_SMD:C_0805_2012Metric
- C2: renamed from C110; footprint valve_pcb_footprints:C_0402_1005Metric -> Capacitor_SMD:C_0402_1005Metric
- R2: renamed from R170; footprint valve_pcb_footprints:R_0603_1608Metric -> Resistor_SMD:R_0603_1608Metric
- R4: renamed from R173; footprint valve_pcb_footprints:R_0603_1608Metric -> Resistor_SMD:R_0603_1608Metric
- R5: renamed from R171; footprint valve_pcb_footprints:R_0603_1608Metric -> Resistor_SMD:R_0603_1608Metric
- R6: renamed from R166; footprint valve_pcb_footprints:R_0603_1608Metric -> Resistor_SMD:R_0603_1608Metric
- R8: renamed from R169; footprint valve_pcb_footprints:R_0603_1608Metric -> Resistor_SMD:R_0603_1608Metric
- renumbered J16 to J2, TP199 to TP1, U32 to U1
Connections:
- net GP16 renamed MISO
- net GP18 renamed SCK
- net GP19 renamed MOSI
- net GP7 renamed SD_CS
Other:
- note removed: "20"
