File: LRUs/User Control Unit/Electrical/User Control Board/user_control_board/user_control_board.kicad_sch (KiCad schematic)
At the start: 0 parts

Commit message: connectors and 5v buck partially done
Changed lines of the file:
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@@
 		)
 	)
-	(text_box "RESPONSIBLE ENGINEER: \nNICHOLAS ALVES\n\nREVIEWERS:"
+	(text_box "RESPONSIBLE ENGINEER: \nNICHOLAS ALVES\nKEVIN LUI\n\nREVIEWERS:"
 		(exclude_from_sim no)
 		(at 171.958 130.048 0)
-		(size 46.99 14.1705)
+		(size 46.99 17.2375)
 		(margins 0.9525 0.9525 0.9525 0.9525)
 		(stroke
