File: LRUs/User Control Unit/Electrical/User Control Board/user_control_board/user_control_board.kicad_pcb (KiCad board)
At the start: 2 copper layers, 88 x 70 mm, 48 parts, among them J16 Micro_SD_Card_Det2, J2 532611071, J3 Screw_Terminal_01x02, SW1 SW_SPDT, U1 TPS62933P, U32 TPD6E05U06RVZ

Commit message: 2 pin connectors added
checking commit
Other:
- copper layers 2 -> 4
Changed lines of the file:
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@@
 	(layers
 		(0 "F.Cu" signal)
+		(4 "In1.Cu" signal)
+		(6 "In2.Cu" signal)
 		(2 "B.Cu" signal)
 		(9 "F.Adhes" user "F.Adhesive")
@@
 	)
 	(setup
+		(stackup
+			(layer "F.SilkS"
+				(type "Top Silk Screen")
+			)
+			(layer "F.Paste"
+				(type "Top Solder Paste")
+			)
+			(layer "F.Mask"
+				(type "Top Solder Mask")
+				(thickness 0.01)
+			)
+			(layer "F.Cu"
+				(type "copper")
+				(thickness 0.035)
+			)
+			(layer "dielectric 1"
+				(type "prepreg")
+				(thickness 0.1)
+				(material "FR4")
+				(epsilon_r 4.5)
+				(loss_tangent 0.02)
+			)
+			(layer "In1.Cu"
+				(type "copper")
+				(thickness 0.035)
+			)
+			(layer "dielectric 2"
+				(type "core")
+				(thickness 1.24)
+				(material "FR4")
+				(epsilon_r 4.5)
+				(loss_tangent 0.02)
+			)
+			(layer "In2.Cu"
+				(type "copper")
+				(thickness 0.035)
+			)
+			(layer "dielectric 3"
+				(type "prepreg")
+				(thickness 0.1)
+				(material "FR4")
+				(epsilon_r 4.5)
+				(loss_tangent 0.02)
+			)
+			(layer "B.Cu"
+				(type "copper")
+				(thickness 0.035)
+			)
+			(layer "B.Mask"
+				(type "Bottom Solder Mask")
+				(thickness 0.01)
+			)
+			(layer "B.Paste"
+				(type "Bottom Solder Paste")
+			)
+			(layer "B.SilkS"
+				(type "Bottom Silk Screen")
+			)
+			(copper_finish "None")
+			(dielectric_constraints no)
+		)
 		(pad_to_mask_clearance 0)
 		(allow_soldermask_bridges_in_footprints no)
@@
 		(capping no)
 		(filling no)
+		(zone_defaults)
 		(pcbplotparams
 			(layerselection 0x00000000_00000000_55555555_5755f5ff)
@@
 		)
 		(sheetname "/LCD Connector/")
+		(sheetfile "lcd_connector.kicad_sch")
 		(units
 			(unit
@@
 		(property ki_fp_filters "C_*")
 		(sheetname "/SD Card/")
+		(sheetfile "sd_card.kicad_sch")
 		(units
 			(unit
@@
 		(property ki_fp_filters "R_*")
 		(sheetname "/SD Card/")
+		(sheetfile "sd_card.kicad_sch")
 		(units
 			(unit
@@
 		(property ki_fp_filters "Pin* Test*")
 		(sheetname "/SD Card/")
+		(sheetfile "sd_card.kicad_sch")
 		(units
 			(unit
@@
 		(property ki_fp_filters "Texas*PUSON*14*")
 		(sheetname "/SD Card/")
+		(sheetfile "sd_card.kicad_sch")
 		(units
 			(unit
@@
 		(property ki_fp_filters "R_*")
 		(sheetname "/SD Card/")
+		(sheetfile "sd_card.kicad_sch")
 		(units
 			(unit
@@
 		(property ki_fp_filters "R_*")
 		(sheetname "/SD Card/")
+		(sheetfile "sd_card.kicad_sch")
 		(units
 			(unit
@@
 		(property ki_fp_filters "MountingHole*Pad*")
 		(sheetname "/Mechanical/")
+		(sheetfile "mechanicak.kicad_sch")
 		(units
 			(unit
@@
 		(property ki_fp_filters "MountingHole*Pad*")
 		(sheetname "/Mechanical/")
+		(sheetfile "mechanicak.kicad_sch")
 		(units
 			(unit
@@
 		(property ki_fp_filters "microSD*")
 		(sheetname "/SD Card/")
+		(sheetfile "sd_card.kicad_sch")
 		(units
 			(unit
@@
 		(property ki_fp_filters "R_*")
 		(sheetname "/SD Card/")
+		(sheetfile "sd_card.kicad_sch")
 		(units
 			(unit
@@
 		(property ki_fp_filters "R_*")
 		(sheetname "/SD Card/")
+		(sheetfile "sd_card.kicad_sch")
 		(units
 			(unit
@@
 		)
 		(sheetname "/Connectors/")
+		(sheetfile "connectors.kicad_sch")
 		(units
 			(unit
@@
 		(property ki_fp_filters "C_*")
 		(sheetname "/SD Card/")
+		(sheetfile "sd_card.kicad_sch")
 		(units
 			(unit
@@
 		(property ki_fp_filters "R_*")
 		(sheetname "/SD Card/")
+		(sheetfile "sd_card.kicad_sch")
 		(units
 			(unit
@@
 		(property ki_fp_filters "RaspberryPi?Pico?Common* RaspberryPi?Pico?W?SMD*")
 		(sheetname "/Raspberry Pi/")
+		(sheetfile "raspberry_pi.kicad_sch")
 		(units
 			(unit
@@
 		(property ki_fp_filters "R_*")
 		(sheetname "/SD Card/")
+		(sheetfile "sd_card.kicad_sch")
 		(units
 			(unit
@@
 		(property ki_fp_filters "MountingHole*Pad*")
 		(sheetname "/Mechanical/")
+		(sheetfile "mechanicak.kicad_sch")
 		(units
 			(unit
@@
 		(property ki_fp_filters "MountingHole*Pad*")
 		(sheetname "/Mechanical/")
+		(sheetfile "mechanicak.kicad_sch")
 		(units
 			(unit
@@
 		(property ki_fp_filters "R_*")
 		(sheetname "/SD Card/")
+		(sheetfile "sd_card.kicad_sch")
 		(units
 			(unit
@@
 		(property ki_fp_filters "TerminalBlock*:*")
 		(sheetname "/Power/")
+		(sheetfile "power.kicad_sch")
 		(units
 			(unit
@@
 		)
 		(sheetname "/Raspberry Pi/")
+		(sheetfile "raspberry_pi.kicad_sch")
 		(units
 			(unit

Commit message: connectors and 5v buck partially done
Parts:
- removed C107: 10uF, valve_pcb_footprints:C_0805_2012Metric
- removed C110: 100nF, valve_pcb_footprints:C_0402_1005Metric
- removed the G*** at (190.1, 101.2)
- removed the G*** at (140.6, 111.5)
- removed J16: Micro_SD_Card_Det2, Connector_Card:microSD_HC_Hirose_DM3AT-SF-PEJM5
- removed R1: 47k, valve_pcb_footprints:R_0603_1608Metric
- removed R165, R166, R167, R168, R170, R171: 0, valve_pcb_footprints:R_0603_1608Metric
- removed R169: 10k, valve_pcb_footprints:R_0603_1608Metric
- removed R173: 22, valve_pcb_footprints:R_0603_1608Metric
- removed R3: 20k, valve_pcb_footprints:R_0603_1608Metric
- removed R7: 68k, valve_pcb_footprints:R_0603_1608Metric
- removed the TP1 at (142.9, 82.0)
- removed U32: TPD6E05U06RVZ, Package_SON:Texas_R-PUSON-N14
- added C10: 1uF, Capacitor_SMD:C_0805_2012Metric, F.Cu at (59.7, 118.8)
- added C11: 1uF, Capacitor_SMD:C_0805_2012Metric, F.Cu at (56.2, 110.8)
- added C12: 10uF, Capacitor_Tantalum_SMD:CP_EIA-3216-18_Kemet-A, F.Cu at (56.7, 108.3)
- added C13: 47uF, Capacitor_SMD:C_1206_3216Metric, F.Cu at (154.7, 92.4)
- added C14: 47uF, Capacitor_SMD:C_1206_3216Metric, F.Cu at (154.7, 95.7)
- added C15: 47uF, Capacitor_SMD:C_1206_3216Metric, F.Cu at (154.7, 99.1)
- added C16: 100nF, Capacitor_SMD:C_0402_1005Metric, F.Cu at (140.7, 109.2)
- added C17: 4.7uF, Capacitor_SMD:C_0805_2012Metric, F.Cu at (154.1, 102.3)
- added C18: 30pF, Capacitor_SMD:C_0201_0603Metric, F.Cu at (143.4, 109.1)
- added C19: 680pF, Capacitor_SMD:C_0201_0603Metric, F.Cu at (143.4, 110.9)
- added C20: 100nF, Capacitor_SMD:C_0402_1005Metric, F.Cu at (140.7, 111.2)
- added C21: 10uF, Capacitor_Tantalum_SMD:CP_EIA-7343-31_Kemet-D, F.Cu at (139.8, 93.6)
- added C22: 10uF, Capacitor_Tantalum_SMD:CP_EIA-7343-31_Kemet-D, F.Cu at (139.8, 99.5)
- added C23: 10uF, Capacitor_Tantalum_SMD:CP_EIA-7343-31_Kemet-D, F.Cu at (139.8, 105.3)
- added C8: 10uF, Capacitor_Tantalum_SMD:CP_EIA-3216-18_Kemet-A, F.Cu at (110.8, 95.5)
- added C9: 10uF, Capacitor_Tantalum_SMD:CP_EIA-3216-18_Kemet-A, F.Cu at (110.8, 91.8)
- added D2: GREEN, LED_SMD:LED_0805_2012Metric, F.Cu at (106.5, 36.5)
- added G***: LOGO, LOGO, F.Cu at (205.0, 69.0)
- added J4: Screw_Terminal_01x02, TerminalBlock_Phoenix:TerminalBlock_Phoenix_MPT-0,5-2-2.54_1x02_P2.54mm_Horizontal, F.Cu at (123.0, 120.5)
- added J5: B2B-XH-A, Connector_JST:JST_XH_B2B-XH-A_1x02_P2.50mm_Vertical, F.Cu at (198.5, 119.5)
- added J6: B2B-XH-A, Connector_JST:JST_XH_B2B-XH-A_1x02_P2.50mm_Vertical, F.Cu at (208.8, 119.5)
- added J7: Conn_02x08_Odd_Even, Connector_PinHeader_2.54mm:PinHeader_2x08_P2.54mm_Vertical, F.Cu at (196.3, 50.0)
- added J8: S12B-PH-K-S, Connector_JST:JST_PH_S12B-PH-K_1x12_P2.00mm_Horizontal, F.Cu at (218.5, 79.5)
- added J9: Screw_Terminal_01x02, TerminalBlock_Phoenix:TerminalBlock_Phoenix_MPT-0,5-2-2.54_1x02_P2.54mm_Horizontal, F.Cu at (190.0, 120.5)
- added L2: 1.2uH, Inductor_SMD:L_Coilcraft_XAL6030-XXX, F.Cu at (151.9, 109.9)
- added R10: 220k, Resistor_SMD:R_0603_1608Metric, F.Cu at (121.2, 112.0)
- added R11: 20k, Resistor_SMD:R_0603_1608Metric, F.Cu at (119.5, 112.0)
- added R12: 9.1k, Resistor_SMD:R_0603_1608Metric, F.Cu at (117.8, 112.0)
- added R13: 51k, Resistor_SMD:R_0603_1608Metric, F.Cu at (116.2, 112.0)
- added R14: 0, Resistor_SMD:R_0603_1608Metric, F.Cu at (114.6, 112.0)
- added R15: 68k, Resistor_SMD:R_0603_1608Metric, F.Cu at (111.0, 111.1)
- added R16: 13k, Resistor_SMD:R_0603_1608Metric, F.Cu at (106.9, 111.1)
- added R17: 2k, Resistor_SMD:R_0603_1608Metric, F.Cu at (101.5, 111.8)
- added R18: 220, Resistor_SMD:R_0603_1608Metric, F.Cu at (47.6, 107.7)
- added R19: 32.4k, Resistor_SMD:R_0603_1608Metric, F.Cu at (149.8, 92.0)
- added R20: 127k, Resistor_SMD:R_0603_1608Metric, F.Cu at (149.8, 94.5)
- added R21: 309k, Resistor_SMD:R_0603_1608Metric, F.Cu at (149.8, 97.0)
- added R22: 1.05M, Resistor_SMD:R_0603_1608Metric, F.Cu at (149.8, 99.5)
- added R23: 100k, Resistor_SMD:R_0603_1608Metric, F.Cu at (149.8, 102.0)
- added R24: 18k, Resistor_SMD:R_0603_1608Metric, F.Cu at (149.8, 104.5)
- added TP10: TestPoint, TestPoint:TestPoint_Pad_D1.0mm, F.Cu at (146.3, 98.3)
- added TP11: TestPoint, TestPoint:TestPoint_Pad_D1.0mm, F.Cu at (146.3, 101.4)
- added TP12: TestPoint, TestPoint:TestPoint_Pad_D1.0mm, F.Cu at (146.3, 104.4)
- added TP6: TestPoint, TestPoint:TestPoint_Pad_D1.0mm, F.Cu at (109.0, 110.4)
- added TP7: TestPoint, TestPoint:TestPoint_Pad_D1.0mm, F.Cu at (87.5, 103.0)
- added TP8: TestPoint, TestPoint:TestPoint_Pad_D1.0mm, F.Cu at (146.3, 92.2)
- added TP9: TestPoint, TestPoint:TestPoint_Pad_D1.0mm, F.Cu at (146.3, 95.3)
- added U2: TPS62933P, Package_TO_SOT_SMD:SOT-583-8, F.Cu at (113.8, 107.2)
- added U3: AMS1117-3.3, Package_TO_SOT_SMD:SOT-223-3_TabPin2, F.Cu at (54.7, 116.3)
- added U4: TPS61089RNRR, Package_DFN_QFN:Texas_VQFN-RNR0011A-11, F.Cu at (137.1, 110.3)
- added U5: ~, footprints:Adafruit PCM510x I2S DAC, F.Cu at (88.0, 76.8)
- added U6: ~, footprints:Ada_Ethernet, F.Cu at (183.0, 85.3)
- A1: footprint Module:RaspberryPi_Pico_W_SMD_HandSolder -> Module:RaspberryPi_Pico_Common_Unspecified
- C1: footprint Capacitor_Tantalum_SMD:CP_EIA-7343-31_Kemet-D -> Capacitor_SMD:C_0805_2012Metric
- C2: value 10uF -> 100nF; footprint Capacitor_Tantalum_SMD:CP_EIA-7343-31_Kemet-D -> Capacitor_SMD:C_0402_1005Metric
- C3, C4: value 100nF -> 10uF; footprint valve_pcb_footprints:C_0402_1005Metric -> Capacitor_Tantalum_SMD:CP_EIA-7343-31_Kemet-D
- C5: footprint valve_pcb_footprints:C_0402_1005Metric -> Capacitor_SMD:C_01005_0402Metric
- C6, C7: value 10uF -> 100nF; footprint Capacitor_Tantalum_SMD:CP_EIA-3216-18_Kemet-A -> Capacitor_SMD:C_0402_1005Metric
- J2: value 532611071 -> Micro_SD_Card_Det2; footprint footprints:CONN_532610001-SD_10_MOL -> Connector_Card:microSD_HC_Hirose_DM3AT-SF-PEJM5
- R2: value 220k -> 0; footprint valve_pcb_footprints:R_0603_1608Metric -> Resistor_SMD:R_0603_1608Metric
- R4: value 9.1k -> 22; footprint valve_pcb_footprints:R_0603_1608Metric -> Resistor_SMD:R_0603_1608Metric
- R5: value 51k -> 0; footprint valve_pcb_footprints:R_0603_1608Metric -> Resistor_SMD:R_0603_1608Metric
- R6: footprint valve_pcb_footprints:R_0603_1608Metric -> Resistor_SMD:R_0603_1608Metric
- R8: value 13k -> 10k; footprint valve_pcb_footprints:R_0603_1608Metric -> Resistor_SMD:R_0603_1608Metric
- R9: value 2k -> 47k; footprint valve_pcb_footprints:R_0603_1608Metric -> Resistor_SMD:R_0603_1608Metric
- U1: value TPS62933P -> TPD6E05U06RVZ; footprint Package_TO_SOT_SMD:SOT-583-8 -> Package_SON:Texas_R-PUSON-N14
- moved J2 87.7 mm to (104.4, 60.2)
- moved D1 64.4 mm to (86.5, 125.0), turned to 0 degrees
- moved J3 63.3 mm to (136.0, 121.0)
- moved TP4 60.9 mm to (88.0, 82.9)
- moved TP5 59.4 mm to (87.1, 95.1)
- moved R9 44.5 mm to (100.3, 92.0), turned to 0 degrees
- moved TP3 42.8 mm to (98.4, 106.6)
- moved C2 41.2 mm to (114.7, 52.0), turned to 0 degrees
- moved L1 40.7 mm to (108.0, 102.8), turned to 90 degrees
- moved C1 40.6 mm to (115.5, 49.5), turned to 0 degrees
- moved TP2 38.0 mm to (104.8, 108.6)
- moved U1 36.8 mm to (115.8, 56.5)
- moved C6 34.5 mm to (111.0, 107.0)
- moved TP1 33.7 mm to (178.0, 40.0)
- moved C7 33.7 mm to (110.5, 98.5), turned to 0 degrees
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- renumbered H3 to H2, H2 to H3, TP199 to TP1
Connections:
- A1 pad 1: unconnected-(A1-GPIO0-Pad1) -> LCD_DC
- A1 pad 10: unconnected-(A1-GPIO7-Pad10) -> SD_CS
- A1 pad 11: unconnected-(A1-GPIO8-Pad11) -> G0_RADIO
- A1 pad 12: unconnected-(A1-GPIO9-Pad12) -> PG
- A1 pad 14: unconnected-(A1-GPIO10-Pad14) -> ARM_STAT
- A1 pad 15: unconnected-(A1-GPIO11-Pad15) -> LAUNCH_STAT
- A1 pad 16: unconnected-(A1-GPIO12-Pad16) -> COOL
- A1 pad 17: unconnected-(A1-GPIO13-Pad17) -> VALVE_ARM
- A1 pad 19: unconnected-(A1-GPIO14-Pad19) -> FILL
- A1 pad 2: unconnected-(A1-GPIO1-Pad2) -> LCD_RESET
- A1 pad 20: unconnected-(A1-GPIO15-Pad20) -> VENT
- A1 pad 21: unconnected-(A1-GPIO16-Pad21) -> MISO
- A1 pad 22: unconnected-(A1-GPIO17-Pad22) -> LCD_CS
- A1 pad 24: unconnected-(A1-GPIO18-Pad24) -> SCK
- A1 pad 25: unconnected-(A1-GPIO19-Pad25) -> MOSI
- A1 pad 26: unconnected-(A1-GPIO20-Pad26) -> ETHERNET_RST
- A1 pad 27: unconnected-(A1-GPIO21-Pad27) -> ETHERNET_IRQ
- A1 pad 29: unconnected-(A1-GPIO22-Pad29) -> ETHERNET_CS
- A1 pad 31: unconnected-(A1-GPIO26_ADC0-Pad31) -> DAC_BCK
- A1 pad 32: unconnected-(A1-GPIO27_ADC1-Pad32) -> DAC_WSEL
- A1 pad 34: unconnected-(A1-GPIO28_ADC2-Pad34) -> DAC_DIN
- A1 pad 36: +3V3 -> unconnected-(A1-3V3-Pad36)
- A1 pad 4: unconnected-(A1-GPIO2-Pad4) -> RADIO_RST
- A1 pad 6: unconnected-(A1-GPIO4-Pad6) -> I2C0_SDA
- A1 pad 7: unconnected-(A1-GPIO5-Pad7) -> I2C0_SCL
- A1 pad 9: unconnected-(A1-GPIO6-Pad9) -> RADIO_CS
- C1 pad 1: /Power/5V/VIN -> +3V3
- C2 pad 1: /Power/5V/VIN -> +3V3
- C3 pad 1: /Power/5V/VIN -> /Power/12V/VIN
- C4 pad 1: /Power/5V/BST -> /Power/12V/VIN
- C4 pad 2: /Power/5V/SW -> GND
- C5 pad 1: +5V -> /Power/12V/VIN
- C6 pad 1: +5V -> /Power/5V/BST
- C6 pad 2: GND -> /Power/5V/SW
- J1 pad 1: unconnected-(J1-VIN-Pad1) -> +3V3
- J1 pad 12: unconnected-(J1-TC_CS-Pad12) -> LCD_CS
- J1 pad 13: unconnected-(J1-SCL-Pad13) -> I2C0_SCL
- J1 pad 14: unconnected-(J1-SDA-Pad14) -> I2C0_SDA
- J1 pad 3: unconnected-(J1-GND-Pad3) -> GND
- J1 pad 4: unconnected-(J1-SCK-Pad4) -> SCK
- J1 pad 5: unconnected-(J1-MOSI-Pad5) -> MOSI
- J1 pad 6: unconnected-(J1-MISO-Pad6) -> RADIO_CS
- J1 pad 7: unconnected-(J1-DC-Pad7) -> LCD_DC
- J1 pad 8: unconnected-(J1-RESET-Pad8) -> LCD_RESET
- J2 pad 1: unconnected-(J2-Pad1) -> Net-(J2-DAT2)
- J2 pad 10: unconnected-(J2-Pad10) -> Net-(J2-DET_A)
- J2 pad 2: unconnected-(J2-Pad2) -> Net-(J2-DAT3/CD)
- J2 pad 3: unconnected-(J2-Pad3) -> Net-(J2-CMD)
- J2 pad 4: unconnected-(J2-Pad4) -> +3V3
- J2 pad 5: unconnected-(J2-Pad5) -> Net-(J2-CLK)
- J2 pad 6: unconnected-(J2-Pad6) -> GND
- J2 pad 7: unconnected-(J2-Pad7) -> Net-(J2-DAT0)
- J2 pad 8: unconnected-(J2-Pad8) -> Net-(J2-DAT1)
- J2 pad 9: unconnected-(J2-Pad9) -> GND
- J3 pad 1: /Power/5V/VIN -> Net-(J3-Pin_1)
- R2 pad 1: Net-(R2-Pad1) -> Net-(J2-DAT1)
- R2 pad 2: /Power/5V/VIN -> MOSI
- R4 pad 1: /Power/5V/VEN -> SCK
- R4 pad 2: Net-(R3-Pad1) -> Net-(J2-CLK)
- R5 pad 1: /Power/5V/VEN -> Net-(J2-DAT0)
- R5 pad 2: GND -> MISO
- R6 pad 1: GND -> Net-(J2-DAT3/CD)
- R6 pad 2: /Power/5V/RT -> SD_CS
- R8 pad 1: /Power/5V/FB -> +3V3
- R8 pad 2: GND -> Net-(J2-DET_A)
- R9 pad 1: Net-(D1-A) -> +3V3
- R9 pad 2: +5V -> PG
- TP2 pad 1: /Power/5V/VIN -> PG
- TP3 pad 1: /Power/5V/VEN -> /Power/12V/VIN
- TP4 pad 1: +5V -> /Power/5V/VEN
- TP5 pad 1: /Power/5V/FB -> +5V
- U1 pad 1: /Power/5V/RT -> unconnected-(U1-NC-Pad1)
- U1 pad 2: /Power/5V/VEN -> unconnected-(U1-NC-Pad2)
- U1 pad 3: /Power/5V/VIN -> unconnected-(U1-NC-Pad3)
- U1 pad 4: GND -> unconnected-(U1-NC-Pad4)
- U1 pad 5: /Power/5V/SW -> GND
- U1 pad 6: /Power/5V/BST -> unconnected-(U1-NC-Pad6)
- U1 pad 7: /Power/5V/5V_MAIN_PG -> unconnected-(U1-NC-Pad7)
- U1 pad 8: /Power/5V/FB -> Net-(J2-DAT1)
Routing:
- net /Power/12V/VIN: track 0.00 -> 18.9 mm
- net +5V: track 0.00 -> 10.1 mm
- net PG: track 0.00 -> 8.68 mm
- net GND: track 0.00 -> 7.22 mm, vias 0 -> 6
- net /Power/5V/SW: track 0.00 -> 6.27 mm
- net /Power/5V/VEN: track 0.00 -> 6.19 mm
- net /Power/5V/FB: track 0.00 -> 4.12 mm
- net /Power/5V/RT: track 0.00 -> 3.17 mm
- net Net-(R11-Pad1): track 0.00 -> 2.32 mm
- net Net-(R10-Pad1): track 0.00 -> 1.71 mm
- net /Power/5V/BST: track 0.00 -> 1.53 mm
- removed copper zone on F.Cu, net GND
Other:
- board size 88 x 70 mm -> 130 x 80 mm
- board text removed: "PEARL"
- board text removed: "REV A"

Commit message: 12 V partially done
Parts:
- moved SW1 114.9 mm to (115.4, 149.3), turned to 0 degrees
- moved R19 81.9 mm to (154.2, 173.8), turned to 90 degrees
- moved C17 69.7 mm to (149.2, 171.8), turned to -90 degrees
- moved R20 69.0 mm to (149.3, 163.4), turned to -90 degrees
- moved TP11 67.8 mm to (139.0, 168.8)
- moved TP10 67.8 mm to (139.0, 165.8)
- moved TP9 67.8 mm to (139.0, 162.7)
- moved C18 61.5 mm to (153.9, 169.8)
- moved C19 61.3 mm to (153.9, 171.2)
- moved TP8 50.1 mm to (139.0, 141.8)
- moved D1 28.7 mm to (91.8, 96.8)
- moved L2 28.5 mm to (126.7, 96.5), turned to 90 degrees
- moved C13 24.5 mm to (131.9, 101.4)
- moved C14 24.2 mm to (131.9, 103.9)
- moved C15 23.9 mm to (131.9, 106.4)
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Connections:
- L1 pad 1: /Power/5V/SW -> +5V
- L1 pad 2: +5V -> /Power/5V/SW
Routing:
- net /Power/12V/VIN: track 18.9 -> 0.54 mm, vias 0 -> 18
- net +5V: track 10.1 -> 0.00 mm, vias 0 -> 9
- net GND: track 7.22 -> 0.00 mm, vias 6 -> 5
- net /Power/5V/SW: track 6.27 -> 0.00 mm
- net /Power/5V/FB: track 4.12 -> 7.40 mm
- added copper zone on F.Cu, net +12V
- added copper zone on F.Cu, net +5V
- added copper zone on F.Cu, net /Power/12V/VIN
- added copper zone on F.Cu, net /Power/5V/SW
- added copper zone on F.Cu, net GND
- added copper zone on F.Cu, net Net-(U4-BOOT)
