File: LRUs/User Control Unit/Electrical/User Interface Board/user_interface_board/block_diagram.kicad_sch (KiCad schematic)
At the start: 0 parts

Commit message: style & add prod files
Other:
- title: (none) -> Block Diagram
Changed lines of the file:
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@@
 	(generator_version "10.0")
 	(paper "A4")
+	(title_block
+		(title "Block Diagram")
+		(date "2026-10-26")
+		(rev "A")
+	)
 	(sheet_instances
 		(path "/"
