File: LRUs/User Control Unit/Electrical/User Interface Board/user_interface_board/user_interface_board.kicad_sch (KiCad schematic)
At the start: 0 parts

Commit message: Commit updates to user interface
Other:
- note added: "EMERALD - REV A"
- note added: "USER INTERFACE BOARD"

Commit message: interface pcb
Changed lines of the file:
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@@
 		)
 	)
-	(text_box "RESPONSIBLE ENGINEER: \nNICHOLAS ALVES\nJAMES F\n\nREVIEWERS:"
+	(text_box "RESPONSIBLE ENGINEER: \nJAMES F\n\nREVIEWERS:\nNICHOLAS ALVES"
 		(exclude_from_sim no)
 		(at 174.498 121.158 0)

Commit message: style & add prod files
Other:
- title: (none) -> Title Page
